File: turboquant_v5/hardware/schematics/analog.kicad_sch (KiCad schematic)
At the start: 70 parts, among them U1 DG408, U2 DG408, U3 OPA1641, U4 OPA1641

Commit message: Update T/R bridge bias resistors: 10k -> 1k
- Fixes insertion loss issue identified in MUR120 analysis
- 1k bias provides ~500uA current for <10dB RX path loss
- 8x bias resistors (R1-R8) changed from 10k to 1k in analog.kicad_sch
- Power dissipation: 25mW per resistor (acceptable)
- See MUR120_TR_BRIDGE_ANALYSIS.md for full calculation
Parts:
- R1, R10, R13, R16, R19, R22, R4, R7: value 10k -> 1k
Changed lines of the file:
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@@
     (uuid "r1-ch0")
     (property "Reference" "R1" (at 67.31 26.67 0) (effects (font (size 1.27 1.27)) (justify left)))
-    (property "Value" "10k" (at 59.69 27.94 0) (effects (font (size 1.27 1.27)) (justify right)))
+    (property "Value" "1k" (at 59.69 27.94 0) (effects (font (size 1.27 1.27)) (justify right)))
     (property "Footprint" "Resistor_SMD:R_0603_1608Metric" (at 63.5 27.94 0) (effects (font (size 1.27 1.27)) hide))
     (pin "1" (uuid "r1-ch0-p1")) (pin "2" (uuid "r1-ch0-p2")))
@@
     (uuid "r1-ch1")
     (property "Reference" "R4" (at 67.31 31.750000000000004 0) (effects (font (size 1.27 1.27)) (justify left)))
-    (property "Value" "10k" (at 59.69 33.02 0) (effects (font (size 1.27 1.27)) (justify right)))
+    (property "Value" "1k" (at 59.69 33.02 0) (effects (font (size 1.27 1.27)) (justify right)))
     (property "Footprint" "Resistor_SMD:R_0603_1608Metric" (at 63.5 27.94 0) (effects (font (size 1.27 1.27)) hide))
     (pin "1" (uuid "r1-ch1-p1")) (pin "2" (uuid "r1-ch1-p2")))
@@
     (uuid "r1-ch2")
     (property "Reference" "R7" (at 67.31 36.83 0) (effects (font (size 1.27 1.27)) (justify left)))
-    (property "Value" "10k" (at 59.69 38.1 0) (effects (font (size 1.27 1.27)) (justify right)))
+    (property "Value" "1k" (at 59.69 38.1 0) (effects (font (size 1.27 1.27)) (justify right)))
     (property "Footprint" "Resistor_SMD:R_0603_1608Metric" (at 63.5 27.94 0) (effects (font (size 1.27 1.27)) hide))
     (pin "1" (uuid "r1-ch2-p1")) (pin "2" (uuid "r1-ch2-p2")))
@@
     (uuid "r1-ch3")
     (property "Reference" "R10" (at 67.31 41.91 0) (effects (font (size 1.27 1.27)) (justify left)))
-    (property "Value" "10k" (at 59.69 43.18 0) (effects (font (size 1.27 1.27)) (justify right)))
+    (property "Value" "1k" (at 59.69 43.18 0) (effects (font (size 1.27 1.27)) (justify right)))
     (property "Footprint" "Resistor_SMD:R_0603_1608Metric" (at 63.5 27.94 0) (effects (font (size 1.27 1.27)) hide))
     (pin "1" (uuid "r1-ch3-p1")) (pin "2" (uuid "r1-ch3-p2")))
@@
     (uuid "r1-ch4")
     (property "Reference" "R13" (at 67.31 46.989999999999995 0) (effects (font (size 1.27 1.27)) (justify left)))
-    (property "Value" "10k" (at 59.69 48.26 0) (effects (font (size 1.27 1.27)) (justify right)))
+    (property "Value" "1k" (at 59.69 48.26 0) (effects (font (size 1.27 1.27)) (justify right)))
     (property "Footprint" "Resistor_SMD:R_0603_1608Metric" (at 63.5 27.94 0) (effects (font (size 1.27 1.27)) hide))
     (pin "1" (uuid "r1-ch4-p1")) (pin "2" (uuid "r1-ch4-p2")))
@@
     (uuid "r1-ch5")
     (property "Reference" "R16" (at 67.31 52.07 0) (effects (font (size 1.27 1.27)) (justify left)))
-    (property "Value" "10k" (at 59.69 53.34 0) (effects (font (size 1.27 1.27)) (justify right)))
+    (property "Value" "1k" (at 59.69 53.34 0) (effects (font (size 1.27 1.27)) (justify right)))
     (property "Footprint" "Resistor_SMD:R_0603_1608Metric" (at 63.5 27.94 0) (effects (font (size 1.27 1.27)) hide))
     (pin "1" (uuid "r1-ch5-p1")) (pin "2" (uuid "r1-ch5-p2")))
@@
     (uuid "r1-ch6")
     (property "Reference" "R19" (at 67.31 57.15 0) (effects (font (size 1.27 1.27)) (justify left)))
-    (property "Value" "10k" (at 59.69 58.42 0) (effects (font (size 1.27 1.27)) (justify right)))
+    (property "Value" "1k" (at 59.69 58.42 0) (effects (font (size 1.27 1.27)) (justify right)))
     (property "Footprint" "Resistor_SMD:R_0603_1608Metric" (at 63.5 27.94 0) (effects (font (size 1.27 1.27)) hide))
     (pin "1" (uuid "r1-ch6-p1")) (pin "2" (uuid "r1-ch6-p2")))
@@
     (uuid "r1-ch7")
     (property "Reference" "R22" (at 67.31 62.23 0) (effects (font (size 1.27 1.27)) (justify left)))
-    (property "Value" "10k" (at 59.69 63.5 0) (effects (font (size 1.27 1.27)) (justify right)))
+    (property "Value" "1k" (at 59.69 63.5 0) (effects (font (size 1.27 1.27)) (justify right)))
     (property "Footprint" "Resistor_SMD:R_0603_1608Metric" (at 63.5 27.94 0) (effects (font (size 1.27 1.27)) hide))
     (pin "1" (uuid "r1-ch7-p1")) (pin "2" (uuid "r1-ch7-p2")))
